Commit message: change dual_ur to dual_ur5

File: dual_ur_description/urdf/dual_ur5.urdf.xacro (robot description, xacro)
@@ -1,7 +1,7 @@
 <?xml version="1.0"?>
 <robot xmlns:xacro="http://wiki.ros.org/xacro" name="dual_ur">
-  <!-- ***************************************************************************************************8 -->
-  <!-- import base -->
-  <link
+  <!-- *************************************************************************************************** -->
+  <!-- import dual_base -->
+   <link
     name="dual_base">
     <visual>
@@ -29,7 +29,8 @@
     </collision>
   </link>
-  <!-- ***************************************************************************************************8 -->
-  <!-- import dual ur arms -->
-  <xacro:include filename="$(find ur_description)/urdf/inc/ur_macro.xacro"/>
+  <!-- *************************************************************************************************** -->
+  <!-- import arms -->
+  <!-- import main macro -->
+   <xacro:include filename="$(find ur_description)/urdf/inc/ur_macro.xacro"/>
   <!-- parameters -->
   <xacro:arg name="joint_limit_params" default="$(find ur_description)/config/ur5/joint_limits.yaml"/>
@@ -68,14 +69,7 @@
     safety_pos_margin="$(arg safety_pos_margin)"
     safety_k_position="$(arg safety_k_position)"/>
-  <!-- ***************************************************************************************************8 -->
-  <!-- import grippers -->
-  <xacro:include filename="$(find robotiq_2f_85_gripper_visualization)/urdf/robotiq_arg2f_85_model_macro.xacro" />
-  <!-- gripper left -->
-  <xacro:robotiq_arg2f_85 prefix="gripper_0_"/>
-  <!-- gripper right -->
-  <xacro:robotiq_arg2f_85 prefix="gripper_1_"/>
-  <!-- ***************************************************************************************************8 -->
+  <!-- *************************************************************************************************** -->
   <!-- setup joints -->
-  <!-- joints between dual_base and arms -->
+  <!-- joint between dual_base and arm -->
   <joint name="dual_base_joint_0" type="fixed">
     <parent link="dual_base" />
@@ -88,14 +82,3 @@
     <origin xyz="0 0.357 0" rpy="${-pi/2} ${pi} 0" />
   </joint>
-  <!-- joints between arm and gripper -->
-  <joint name="arm_0_gripper_0_joint" type="fixed">
-    <parent link="arm_0_tool0" />
-    <child link="gripper_0_robotiq_arg2f_base_link" />
-    <origin xyz="0 0 0" rpy="0 0 0" />
-  </joint>
-  <joint name="arm_1_gripper_1_joint" type="fixed">
-    <parent link="arm_1_tool0" />
-    <child link="gripper_1_robotiq_arg2f_base_link" />
-    <origin xyz="0 0 0" rpy="0 0 0" />
-  </joint>
 </robot>
