Commit message: add tcp links

File: dual_ur_description/urdf/dual_ur5_robotiq2f85.urdf.xacro (robot description, xacro)
@@ -44,3 +44,17 @@
     <origin xyz="0 0 0" rpy="0 0 0" />
   </joint>
+  <!-- *************************************************************************************************** -->
+  <!-- add dual arm tcp links (the middle of the gripper fingers) -->
+  <link name="arm_0_tcp"/>
+  <joint name="arm_0_tool0_tcp" type="fixed">
+      <origin xyz="0 0 0.145" rpy="${pi} 0 ${pi/2.0}"/>
+      <parent link="arm_0_tool0"/>
+      <child link="arm_0_tcp"/>
+  </joint>
+  <link name="arm_1_tcp"/>
+  <joint name="arm_1_tool0_tcp" type="fixed">
+      <origin xyz="0 0 0.145" rpy="${pi} 0 ${pi/2.0}"/>
+      <parent link="arm_1_tool0"/>
+      <child link="arm_1_tcp"/>
+  </joint>
 </robot>
