Commit message: update

File: dual_ur_description/urdf/dual_ur5_real.urdf.xacro (robot description, xacro)
@@ -78,8 +78,13 @@
     <origin xyz="0 -0.357 0" rpy="${pi/2} 0 0" />
   </joint>
+  <!-- <joint name="dual_base_joint_1" type="fixed">
+    <parent link="dual_base" />
+    <child link="arm_1_base_link" />
+    <origin xyz="0 0.357 0" rpy="${-pi/2} ${pi} 0" />
+  </joint> -->
   <joint name="dual_base_joint_1" type="fixed">
     <parent link="dual_base" />
     <child link="arm_1_base_link" />
-    <origin xyz="0 0.357 0" rpy="${-pi/2} ${pi} 0" />
+    <origin xyz="-0.00286359  0.3585708  -0.01326747" rpy="1.58859659 0.01214445 3.12246477" />
   </joint>
 </robot>

File: dual_ur_description/urdf/dual_ur5_robotiq2f85_v2.urdf.xacro (robot description, xacro)
@@ -3,5 +3,5 @@
   <!-- *************************************************************************************************** -->
   <!-- import dual_ur5 -->
-  <xacro:include filename="$(find dual_ur_description)/urdf/dual_ur5.urdf.xacro"/>
+  <xacro:include filename="$(find dual_ur_description)/urdf/dual_ur5_real.urdf.xacro"/>
   <!-- parameters -->
    <xacro:arg name="joint_limit_params" default="$(find ur_description)/config/ur5/joint_limits.yaml"/>
@@ -38,10 +38,10 @@
     <parent link="arm_0_tool0" />
     <child link="gripper_0_base_link" />
-    <origin xyz="0 0 0" rpy="0 0 ${pi/2.0}" />
+    <origin xyz="0 0 0.018" rpy="0 0 ${pi/2.0}" />
   </joint>
   <joint name="arm_1_gripper_1_joint" type="fixed">
     <parent link="arm_1_tool0" />
     <child link="gripper_1_base_link" />
-    <origin xyz="0 0 0" rpy="0 0 ${pi/2.0}" />
+    <origin xyz="0 0 0.018" rpy="0 0 ${pi/2.0}" />
   </joint>
   <!-- *************************************************************************************************** -->
@@ -49,5 +49,5 @@
   <link name="arm_0_tcp"/>
   <joint name="arm_0_tool0_tcp" type="fixed">
-      <origin xyz="0 0 0.145" rpy="${pi} 0 0"/>
+      <origin xyz="0 0 0.177" rpy="${pi} 0 0"/>
       <parent link="arm_0_tool0"/>
       <child link="arm_0_tcp"/>
@@ -55,5 +55,5 @@
   <link name="arm_1_tcp"/>
   <joint name="arm_1_tool0_tcp" type="fixed">
-      <origin xyz="0 0 0.145" rpy="${pi} 0 ${pi}"/>
+      <origin xyz="0 0 0.177" rpy="${pi} 0 ${pi}"/>
       <parent link="arm_1_tool0"/>
       <child link="arm_1_tcp"/>
